File: test_kicad_project/mcu.kicad_sch (KiCad schematic)
At the start: 26 parts, among them J10 FTSH-107-01-L-DV-K, J8 Conn_01x03, Q2 BC847, SW2 GT-TC045A-H036-L1A, SW3 GT-TC045A-H036-L1A, U7 STM32F405RGT6, Y2 X322516MLB4SI

Commit message: test_project: update with new mistakes
Parts:
- D1: footprint LED_SMD:LED_0603_1608Metric -> LED_SMD:LED_0402_1005Metric
Connections:
- net +3.3V: now also R8.1; no longer R10.1
- net GND: no longer R8.1
Changed lines of the file:
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@@
 		)
 		(instances
-			(project ""
+			(project "slot-rs232-pi-hat"
 				(path "/e63e39d7-6ac0-4ffd-8aa3-1841a4541b55/bf019eb6-7286-41f0-8b10-b30b6283300c"
 					(reference "Q2")
@@
 		)
 		(instances
-			(project ""
+			(project "slot-rs232-pi-hat"
 				(path "/e63e39d7-6ac0-4ffd-8aa3-1841a4541b55/bf019eb6-7286-41f0-8b10-b30b6283300c"
 					(reference "#PWR010")
@@
 		)
 		(instances
-			(project ""
+			(project "slot-rs232-pi-hat"
 				(path "/e63e39d7-6ac0-4ffd-8aa3-1841a4541b55/bf019eb6-7286-41f0-8b10-b30b6283300c"
 					(reference "J8")
@@
 		)
 		(instances
-			(project ""
+			(project "slot-rs232-pi-hat"
 				(path "/e63e39d7-6ac0-4ffd-8aa3-1841a4541b55/bf019eb6-7286-41f0-8b10-b30b6283300c"
 					(reference "#PWR013")
@@
 		)
 		(instances
-			(project ""
+			(project "slot-rs232-pi-hat"
 				(path "/e63e39d7-6ac0-4ffd-8aa3-1841a4541b55/bf019eb6-7286-41f0-8b10-b30b6283300c"
 					(reference "SW2")
@@
 	(symbol
 		(lib_id "power:+3.3V")
+		(at 66.04 54.61 90)
+		(unit 1)
+		(exclude_from_sim no)
+		(in_bom yes)
+		(on_board yes)
+		(dnp no)
+		(fields_autoplaced yes)
+		(property "Reference" "#PWR017"
+			(at 69.85 54.61 0)
+			(effects
+				(font
+					(size 1.27 1.27)
+				)
+				(hide yes)
+			)
+		)
+		(property "Value" "+3.3V"
+			(at 62.23 54.6099 90)
+			(effects
+				(font
+					(size 1.27 1.27)
+				)
+				(justify left)
+			)
+		)
+		(property "Footprint" ""
+			(at 66.04 54.61 0)
+			(effects
+				(font
+					(size 1.27 1.27)
+				)
+				(hide yes)
+			)
+		)
+		(property "Datasheet" ""
+			(at 66.04 54.61 0)
+			(effects
+				(font
+					(size 1.27 1.27)
+				)
+				(hide yes)
+			)
+		)
+		(property "Description" "Power symbol creates a global label with name \"+3.3V\""
+			(at 66.04 54.61 0)
+			(effects
+				(font
+					(size 1.27 1.27)
+				)
+				(hide yes)
+			)
+		)
+		(pin "1"
+		)
+		(instances
+			(project "slot-rs232-pi-hat"
+				(path "/e63e39d7-6ac0-4ffd-8aa3-1841a4541b55/bf019eb6-7286-41f0-8b10-b30b6283300c"
+					(reference "#PWR017")
+					(unit 1)
+				)
+			)
+		)
+	)
+	(symbol
+		(lib_id "power:+3.3V")
 		(at 80.01 44.45 0)
 		(unit 1)
@@
 		)
 		(instances
-			(project ""
+			(project "slot-rs232-pi-hat"
 				(path "/e63e39d7-6ac0-4ffd-8aa3-1841a4541b55/bf019eb6-7286-41f0-8b10-b30b6283300c"
 					(reference "C1")
@@
 			)
 		)
-		(property "Footprint" "LED_SMD:LED_0603_1608Metric"
+		(property "Footprint" "LED_SMD:LED_0402_1005Metric"
 			(at 161.29 67.31 0)
 			(effects
@@
 		)
 		(instances
-			(project ""
+			(project "slot-rs232-pi-hat"
 				(path "/e63e39d7-6ac0-4ffd-8aa3-1841a4541b55/bf019eb6-7286-41f0-8b10-b30b6283300c"
 					(reference "Y2")
@@
 		)
 		(instances
-			(project ""
+			(project "slot-rs232-pi-hat"
 				(path "/e63e39d7-6ac0-4ffd-8aa3-1841a4541b55/bf019eb6-7286-41f0-8b10-b30b6283300c"
 					(reference "R7")
@@
 		)
 		(instances
-			(project ""
-				(path "/e63e39d7-6ac0-4ffd-8aa3-1841a4541b55/bf019eb6-7286-41f0-8b10-b30b6283300c"
-					(reference "J10")
-					(unit 1)
-				)
-			)
-		)
-	)
-	(symbol
-		(lib_id "power:+3.3V")
-		(at 190.5 100.33 0)
-		(unit 1)
-		(exclude_from_sim no)
-		(in_bom yes)
-		(on_board yes)
-		(dnp no)
-		(fields_autoplaced yes)
-		(property "Reference" "#PWR023"
-			(at 190.5 104.14 0)
-			(effects
-				(font
-					(size 1.27 1.27)
-				)
-				(hide yes)
-			)
-		)
-		(property "Value" "+3.3V"
-			(at 190.5 95.25 0)
-			(effects
-				(font
-					(size 1.27 1.27)
-				)
-			)
-		)
-		(property "Footprint" ""
-			(at 190.5 100.33 0)
-			(effects
-				(font
-					(size 1.27 1.27)
-				)
-				(hide yes)
-			)
-		)
-		(property "Datasheet" ""
-			(at 190.5 100.33 0)
-			(effects
-				(font
-					(size 1.27 1.27)
-				)
-				(hide yes)
-			)
-		)
-		(property "Description" "Power symbol creates a global label with name \"+3.3V\""
-			(at 190.5 100.33 0)
-			(effects
-				(font
-					(size 1.27 1.27)
-				)
-				(hide yes)
-			)
-		)
-		(pin "1"
-		)
-		(instances
 			(project "slot-rs232-pi-hat"
 				(path "/e63e39d7-6ac0-4ffd-8aa3-1841a4541b55/bf019eb6-7286-41f0-8b10-b30b6283300c"
-					(reference "#PWR023")
+					(reference "J10")
 					(unit 1)
 				)
@@
 	(symbol
 		(lib_id "power:GND")
-		(at 66.04 54.61 270)
-		(unit 1)
-		(exclude_from_sim no)
-		(in_bom yes)
-		(on_board yes)
-		(dnp no)
-		(fields_autoplaced yes)
-		(property "Reference" "#PWR017"
-			(at 59.69 54.61 0)
-			(effects
-				(font
-					(size 1.27 1.27)
-				)
-				(hide yes)
-			)
-		)
-		(property "Value" "GND"
-			(at 62.23 54.6099 90)
-			(effects
-				(font
-					(size 1.27 1.27)
-				)
-				(justify right)
-			)
-		)
-		(property "Footprint" ""
-			(at 66.04 54.61 0)
-			(effects
-				(font
-					(size 1.27 1.27)
-				)
-				(hide yes)
-			)
-		)
-		(property "Datasheet" ""
-			(at 66.04 54.61 0)
-			(effects
-				(font
-					(size 1.27 1.27)
-				)
-				(hide yes)
-			)
-		)
-		(property "Description" "Power symbol creates a global label with name \"GND\" , ground"
-			(at 66.04 54.61 0)
-			(effects
-				(font
-					(size 1.27 1.27)
-				)
-				(hide yes)
-			)
-		)
-		(pin "1"
-		)
-		(instances
-			(project "slot-rs232-pi-hat"
-				(path "/e63e39d7-6ac0-4ffd-8aa3-1841a4541b55/bf019eb6-7286-41f0-8b10-b30b6283300c"
-					(reference "#PWR017")
-					(unit 1)
-				)
-			)
-		)
-	)
-	(symbol
-		(lib_id "power:GND")
 		(at 60.96 76.2 0)
 		(unit 1)
@@
 		)
 		(instances
-			(project ""
+			(project "slot-rs232-pi-hat"
 				(path "/e63e39d7-6ac0-4ffd-8aa3-1841a4541b55/bf019eb6-7286-41f0-8b10-b30b6283300c"
 					(reference "#PWR012")
