File: test_kicad_project/power_supply.kicad_sch (KiCad schematic)
At the start: 28 parts, among them J2 XDJK-0051-025, J5 ZX-5557-4.2-2-2PWZ, J6 ZX-5557-4.2-2-2PWZ, Q1 Si2319CDS, SW1 SK-3296S-01-L1, U4 TPS54531DDAR, U6 LD1117S33TR

Commit message: test_project: update with new mistakes
Parts:
- R3: value 1.96k -> 10k
Changed lines of the file:
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@@
 		)
 		(instances
-			(project ""
+			(project "slot-rs232-pi-hat"
 				(path "/e63e39d7-6ac0-4ffd-8aa3-1841a4541b55/db941ee9-9dec-49e9-80b2-8ef11bdcef9f"
 					(reference "#PWR05")
@@
 		)
 		(instances
-			(project ""
+			(project "slot-rs232-pi-hat"
 				(path "/e63e39d7-6ac0-4ffd-8aa3-1841a4541b55/db941ee9-9dec-49e9-80b2-8ef11bdcef9f"
 					(reference "Q1")
@@
 		)
 		(instances
-			(project ""
+			(project "slot-rs232-pi-hat"
 				(path "/e63e39d7-6ac0-4ffd-8aa3-1841a4541b55/db941ee9-9dec-49e9-80b2-8ef11bdcef9f"
 					(reference "D4")
@@
 		)
 		(instances
-			(project ""
+			(project "slot-rs232-pi-hat"
 				(path "/e63e39d7-6ac0-4ffd-8aa3-1841a4541b55/db941ee9-9dec-49e9-80b2-8ef11bdcef9f"
 					(reference "#PWR043")
@@
 		)
 		(instances
-			(project ""
+			(project "slot-rs232-pi-hat"
 				(path "/e63e39d7-6ac0-4ffd-8aa3-1841a4541b55/db941ee9-9dec-49e9-80b2-8ef11bdcef9f"
 					(reference "C13")
@@
 		)
 		(instances
-			(project ""
+			(project "slot-rs232-pi-hat"
 				(path "/e63e39d7-6ac0-4ffd-8aa3-1841a4541b55/db941ee9-9dec-49e9-80b2-8ef11bdcef9f"
 					(reference "SW1")
@@
 			)
 		)
-		(property "Value" "1.96k"
+		(property "Value" "10k"
 			(at 208.28 57.1499 0)
 			(effects
@@
 		)
 		(instances
-			(project ""
+			(project "slot-rs232-pi-hat"
 				(path "/e63e39d7-6ac0-4ffd-8aa3-1841a4541b55/db941ee9-9dec-49e9-80b2-8ef11bdcef9f"
 					(reference "L1")
@@
 		)
 		(instances
-			(project ""
+			(project "slot-rs232-pi-hat"
 				(path "/e63e39d7-6ac0-4ffd-8aa3-1841a4541b55/db941ee9-9dec-49e9-80b2-8ef11bdcef9f"
 					(reference "C18")
@@
 		)
 		(instances
-			(project ""
+			(project "slot-rs232-pi-hat"
 				(path "/e63e39d7-6ac0-4ffd-8aa3-1841a4541b55/db941ee9-9dec-49e9-80b2-8ef11bdcef9f"
 					(reference "#PWR031")
@@
 		)
 		(instances
-			(project ""
+			(project "slot-rs232-pi-hat"
 				(path "/e63e39d7-6ac0-4ffd-8aa3-1841a4541b55/db941ee9-9dec-49e9-80b2-8ef11bdcef9f"
 					(reference "U4")
@@
 		)
 		(instances
-			(project ""
+			(project "slot-rs232-pi-hat"
 				(path "/e63e39d7-6ac0-4ffd-8aa3-1841a4541b55/db941ee9-9dec-49e9-80b2-8ef11bdcef9f"
 					(reference "C14")
@@
 		)
 		(instances
-			(project ""
+			(project "slot-rs232-pi-hat"
 				(path "/e63e39d7-6ac0-4ffd-8aa3-1841a4541b55/db941ee9-9dec-49e9-80b2-8ef11bdcef9f"
 					(reference "D13")
@@
 		)
 		(instances
-			(project ""
+			(project "slot-rs232-pi-hat"
 				(path "/e63e39d7-6ac0-4ffd-8aa3-1841a4541b55/db941ee9-9dec-49e9-80b2-8ef11bdcef9f"
 					(reference "R1")
