File: test_kicad_project/slot-rs232-pi-hat.kicad_sch (KiCad schematic)
At the start: 2 parts, among them J1 ZHOURI 2.54-2*20, J7 Conn_01x03

Commit message: test_project: update with new mistakes
Other:
- moved on the sheet: J1, J7
